Commit message: [feat, fix] agconav_description 드론 모델 추가 및 시뮬레이션 구동 오류 수정

File: config/clearpath_a300/robot.urdf.xacro (robot description, xacro)
@@ -22,4 +22,9 @@
   <!-- Mounts -->
   <!-- Sensors -->
+  <!-- lidar3d_0 -->
+  <xacro:include filename="$(find clearpath_sensors_description)/urdf/ouster_os1.urdf.xacro"/>
+  <xacro:ouster_os1 name="lidar3d_0" parent_link="base_link" min_ang_h="-3.141592" max_ang_h="3.141592" min_ang_v="-0.261799" max_ang_v="0.261799" min_range="0.9" max_range="130.0" update_rate="20" samples_h="1024" samples_v="64" base="base" cap="halo">
+    <origin xyz="0.0 0.0 0.5" rpy="0.0 0.0 0.0"/>
+  </xacro:ouster_os1>
   <!-- imu_0 -->
   <xacro:include filename="$(find clearpath_sensors_description)/urdf/phidgets_spatial.urdf.xacro"/>
@@ -27,4 +32,9 @@
     <origin xyz="0.059 0.0 0.161275" rpy="0.0 0.0 0.0"/>
   </xacro:phidgets_spatial>
+  <!-- gps_0 -->
+  <xacro:include filename="$(find clearpath_sensors_description)/urdf/novatel_smart7.urdf.xacro"/>
+  <xacro:novatel_smart7 name="gps_0" parent_link="base_link">
+    <origin xyz="-0.15 0.0 0.45" rpy="0.0 0.0 0.0"/>
+  </xacro:novatel_smart7>
   <!-- Manipulators -->
   <!-- Extras -->

Commit message: [feat] sim: 멀티로봇 센서 정렬 및 Go2 초기 자세 안정화

File: config/clearpath_a300/robot.urdf.xacro (robot description, xacro)
@@ -25,15 +25,15 @@
   <xacro:include filename="$(find clearpath_sensors_description)/urdf/ouster_os1.urdf.xacro"/>
   <xacro:ouster_os1 name="lidar3d_0" parent_link="base_link" min_ang_h="-3.141592" max_ang_h="3.141592" min_ang_v="-0.261799" max_ang_v="0.261799" min_range="0.9" max_range="130.0" update_rate="20" samples_h="1024" samples_v="64" base="base" cap="halo">
-    <origin xyz="0.0 0.0 0.5" rpy="0.0 0.0 0.0"/>
+    <origin xyz="0.0 0.0 0.23" rpy="0.0 0.0 0.0"/>
   </xacro:ouster_os1>
   <!-- imu_0 -->
   <xacro:include filename="$(find clearpath_sensors_description)/urdf/phidgets_spatial.urdf.xacro"/>
   <xacro:phidgets_spatial name="imu_0" parent_link="base_link">
-    <origin xyz="0.059 0.0 0.161275" rpy="0.0 0.0 0.0"/>
+    <origin xyz="-0.1 0.0 0.202259" rpy="0.0 0.0 0.0"/>
   </xacro:phidgets_spatial>
   <!-- gps_0 -->
   <xacro:include filename="$(find clearpath_sensors_description)/urdf/novatel_smart7.urdf.xacro"/>
   <xacro:novatel_smart7 name="gps_0" parent_link="base_link">
-    <origin xyz="-0.15 0.0 0.45" rpy="0.0 0.0 0.0"/>
+    <origin xyz="-0.15 0.0 0.242259" rpy="0.0 0.0 0.0"/>
   </xacro:novatel_smart7>
   <!-- Manipulators -->

File: src/agconav_description/urdf/leg/leg_sensors.xacro (robot description, xacro)
@@ -22,5 +22,5 @@
       <parent link="${parent}"/>
       <child link="os1_lidar"/>
-      <origin xyz="0.0 0.0 0.12" rpy="0 0 0"/>
+      <origin xyz="0.0 0.0 0.09385" rpy="0 0 0"/>
     </joint>
     <!-- ===== GPS ===== -->
@@ -35,5 +35,5 @@
       <parent link="${parent}"/>
       <child link="gps_link"/>
-      <origin xyz="-0.08 0.0 0.10" rpy="0 0 0"/>
+      <origin xyz="-0.10 0.0 0.068" rpy="0 0 0"/>
     </joint>
     <!-- ===== Gazebo 센서 정의 ===== -->
@@ -62,4 +62,5 @@
     <gazebo reference="${parent}">
       <sensor name="leg_imu_sensor" type="imu">
+        <pose>0 0 -0.025 0 0 0</pose>
         <topic>${ns}/imu</topic>
         <gz_frame_id>${parent}</gz_frame_id>

File: src/agconav_description/urdf/leg/leg_with_sensors.urdf.xacro (robot description, xacro)
@@ -7,5 +7,5 @@
   <xacro:include filename="$(find unitree_go2_description)/urdf/unitree_go2_robot.xacro"/>
   <!-- AG-CoNav 센서 오버레이 매크로 -->
-  <xacro:include filename="$(find agconav_description)/urdf/leg_sensors.xacro"/>
+  <xacro:include filename="$(find agconav_description)/urdf/leg/leg_sensors.xacro"/>
   <!-- base_link 에 leg 네임스페이스로 센서 부착 -->
   <xacro:leg_sensors parent="base_link" ns="leg"/>

Commit message: Jongheon 시뮬레이션 환경 세팅 (#6)
* Update CONTRIBUTING.md

* CONTRIBUTING.md 수정: 고정사항

* fix: readme, file

* [docx] README.md 수정

* [FEAT] X3, A300, husky 로봇 모델 및 생성 설정 추가

* docx: README.md 최신화

* feat: unitree_go2_ros2_jazzy를 vcstool 외부 의존성으로 전환

* [FEAT, DOCX] 시뮬레이션 로드, README수정

* [docx] README.md, CONTRIBUTING.md 수정

* [feat]: Nav2 골격 lauch에 넣기, 월드에 datum + 센서 시스템 플러그인

* [feat, fix] agconav_description 드론 모델 추가 및 시뮬레이션 구동 오류 수정

* [docx] 팀원들을 위한 시뮬레이션 가이드북 제작

* [feat] 각 로봇에 센서 부착 및 센서가 겹치는 부분 수정

* [feat] 센서 토픽을 각 파트가 정한  이름으로 변경

* [docx] CONTRIBUTING.md에 datum 내용 적용

* [feat] sim: 멀티로봇 센서 정렬 및 Go2 초기 자세 안정화

File: config/clearpath_a300/robot.urdf.xacro (robot description, xacro)
@@ -22,9 +22,19 @@
   <!-- Mounts -->
   <!-- Sensors -->
+  <!-- lidar3d_0 -->
+  <xacro:include filename="$(find clearpath_sensors_description)/urdf/ouster_os1.urdf.xacro"/>
+  <xacro:ouster_os1 name="lidar3d_0" parent_link="base_link" min_ang_h="-3.141592" max_ang_h="3.141592" min_ang_v="-0.261799" max_ang_v="0.261799" min_range="0.9" max_range="130.0" update_rate="20" samples_h="1024" samples_v="64" base="base" cap="halo">
+    <origin xyz="0.0 0.0 0.23" rpy="0.0 0.0 0.0"/>
+  </xacro:ouster_os1>
   <!-- imu_0 -->
   <xacro:include filename="$(find clearpath_sensors_description)/urdf/phidgets_spatial.urdf.xacro"/>
   <xacro:phidgets_spatial name="imu_0" parent_link="base_link">
-    <origin xyz="0.059 0.0 0.161275" rpy="0.0 0.0 0.0"/>
+    <origin xyz="-0.1 0.0 0.202259" rpy="0.0 0.0 0.0"/>
   </xacro:phidgets_spatial>
+  <!-- gps_0 -->
+  <xacro:include filename="$(find clearpath_sensors_description)/urdf/novatel_smart7.urdf.xacro"/>
+  <xacro:novatel_smart7 name="gps_0" parent_link="base_link">
+    <origin xyz="-0.15 0.0 0.242259" rpy="0.0 0.0 0.0"/>
+  </xacro:novatel_smart7>
   <!-- Manipulators -->
   <!-- Extras -->
